File: Highz-stereo.kicad_pcb (KiCad board)
At the start: 2 copper layers, 62.5 x 97.5 mm, 79 parts, among them J1 Conn_01x01_Female, J10 Conn_01x01_Female, J11 Conn_01x01_Female, J12 Conn_01x01_Female, J13 Potmeter ground A, J14 potmeter ground B, J16 Conn_01x01_Female, J17 Conn_01x01_Female, J18 Conn_01x01_Female, J19 Conn_01x01_Female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

Commit message: Add files via upload
Parts:
- removed U1, U3: L7812CV, Package_TO_SOT_THT:TO-220-3_Vertical
- added D1: ZPD11, Diode_THT:D_DO-35_SOD27_P10.16mm_Horizontal, F.Cu at (79.3, 52.5)
- added D10: ZPD11, Diode_THT:D_DO-35_SOD27_P10.16mm_Horizontal, F.Cu at (51.3, 52.5)
- added R1: 100, Resistor_THT:R_Axial_DIN0204_L3.6mm_D1.6mm_P5.08mm_Horizontal, F.Cu at (92.5, 64.0)
- added R23: 100, Resistor_THT:R_Axial_DIN0204_L3.6mm_D1.6mm_P5.08mm_Horizontal, F.Cu at (65.0, 64.0)
- added R27: 150, Resistor_THT:R_Axial_DIN0204_L3.6mm_D1.6mm_P5.08mm_Horizontal, F.Cu at (51.6, 113.0)
- added R28: 150, Resistor_THT:R_Axial_DIN0204_L3.6mm_D1.6mm_P5.08mm_Horizontal, F.Cu at (73.0, 113.0)
- C21, C22: value 0.33uF -> 680pF
- J13: value Potmeter ground A -> potmeter ground B
- J14: value potmeter ground B -> Potmeter ground A
- U2: value OPA4134 -> OPA1679
- moved C21 59.2 mm to (59.8, 113.0)
- moved C22 59.1 mm to (86.0, 113.0)
- moved J13 33.5 mm to (89.5, 91.0)
- moved J14 28.5 mm to (56.0, 91.0)
- moved C11 6.36 mm to (86.5, 108.0)
- moved C8 6.36 mm to (62.0, 108.5)
- moved R10 3.50 mm to (62.6, 104.5)
- moved R2 3.50 mm to (49.5, 104.5)
- moved D2 3.00 mm to (46.5, 99.0)
- moved D3 3.00 mm to (59.0, 99.0)
- moved D4 3.00 mm to (46.4, 95.0)
- moved D5 3.00 mm to (59.0, 95.0)
- moved D6 3.00 mm to (73.2, 98.5)
- moved D7 3.00 mm to (84.9, 98.5)
- moved D8 3.00 mm to (73.2, 95.0)
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Connections:
- C21 pad 1: Net-(U1-IN) -> ind
- C21 pad 2: GND -> Net-(C21-Pad2)
- C22 pad 1: Net-(U3-IN) -> indR
- C22 pad 2: V-R -> Net-(C22-Pad2)
- J13 pad 1: V- -> V-R
- J14 pad 1: V-R -> V-
- R25 pad 1: Net-(U3-IN) -> Net-(D1-K)
- R26 pad 1: Net-(U3-IN) -> Net-(D1-K)
- R5 pad 1: Net-(U1-IN) -> Net-(D10-K)
- R6 pad 1: Net-(U1-IN) -> Net-(D10-K)
Routing:
- net Net-(D10-K): track 0.00 -> 44.9 mm
- net Net-(D1-K): track 0.00 -> 35.7 mm
- net Net-(U1-IN): track 35.0 -> 0.00 mm
- net Net-(U3-IN): track 29.4 -> 0.00 mm
- net Net-(C22-Pad2): track 0.00 -> 16.7 mm
- net Net-(U2D--): track 49.7 -> 33.1 mm
- net VCCR: track 85.2 -> 72.7 mm
- net VCC: track 96.9 -> 84.8 mm
- net Net-(C21-Pad2): track 0.00 -> 11.8 mm
- net V-: track 127.3 -> 132.4 mm, vias 1 -> 0
- net indR: track 59.0 -> 63.2 mm
- net Net-(C17-Pad2): track 49.7 -> 53.7 mm
- net Net-(C10-Pad1): track 19.4 -> 23.3 mm
- net GND: track 18.4 -> 14.5 mm
- net ind: track 56.4 -> 59.7 mm
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Other:
- board text added: "IN B"

Commit message: Add files via upload
Parts:
- removed C18: 33uF, Capacitor_THT:C_Disc_D5.0mm_W2.5mm_P2.50mm
- added C23: 33uF, Capacitor_THT:CP_Radial_D5.0mm_P2.00mm, F.Cu at (63.5, 86.0)
- C11, C16, C19, C2, C20, C4, C5, C8: footprint Capacitor_THT:C_Disc_D5.0mm_W2.5mm_P2.50mm -> Capacitor_THT:C_Rect_L18.0mm_W9.0mm_P15.00mm_FKS3_FKP3
- C14, C17, C6, C9: footprint Capacitor_THT:C_Disc_D5.0mm_W2.5mm_P2.50mm -> Capacitor_THT:C_Rect_L7.2mm_W4.5mm_P5.00mm_FKS2_FKP2_MKS2_MKP2
- C21, C22: footprint Capacitor_THT:C_Disc_D5.0mm_W2.5mm_P2.50mm -> Capacitor_THT:C_Rect_L7.0mm_W4.5mm_P5.00mm
- C3: footprint Capacitor_THT:C_Disc_D5.0mm_W2.5mm_P2.50mm -> Capacitor_THT:CP_Radial_D5.0mm_P2.00mm
- moved C3 35.4 mm to (75.0, 86.0), turned to 0 degrees
- moved D10 29.6 mm to (62.0, 80.1), turned to 90 degrees
- moved D1 27.9 mm to (75.5, 80.2), turned to 90 degrees
- moved C21 17.7 mm to (43.5, 106.0), turned to -90 degrees
- moved C4 16.5 mm to (63.0, 60.0)
- moved R27 15.3 mm to (66.5, 109.5), turned to -90 degrees
- moved C2 13.5 mm to (43.0, 60.0)
- moved C5 13.5 mm to (53.0, 60.0)
- moved C1 12.9 mm to (51.0, 67.0), turned to 180 degrees
- moved C20 11.9 mm to (94.5, 45.0)
- moved C22 10.5 mm to (96.5, 112.0), turned to 90 degrees
- moved C16 10.5 mm to (74.5, 60.0)
- moved R8 10.5 mm to (58.5, 64.0)
- moved C11 10.0 mm to (76.5, 108.5)
- moved C19 10.0 mm to (84.5, 60.0)
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Connections:
- C3 pad 1: VCC -> VCCR
- C3 pad 2: GND -> V-R
Routing:
- net indR: track 63.2 -> 127.1 mm, vias 0 -> 1
- net GND: track 14.5 -> 57.1 mm
- net V-R: track 117.9 -> 154.9 mm
- net Net-(D4-A): track 56.2 -> 89.6 mm
- net Net-(C4-Pad2): track 7.62 -> 38.8 mm
- net Net-(C14-Pad2): track 31.9 -> 58.6 mm, vias 1 -> 0
- net Net-(C17-Pad2): track 53.7 -> 79.2 mm, vias 0 -> 1
- net /2A: track 30.1 -> 48.3 mm
- net V-: track 132.4 -> 149.9 mm
- net ind: track 59.7 -> 74.8 mm
- net /3: track 37.8 -> 51.1 mm
- net Net-(C5-Pad2): track 8.04 -> 21.2 mm
- net Net-(C19-Pad2): track 13.2 -> 26.3 mm
- net Net-(C11-Pad1): track 26.0 -> 38.9 mm
- net Net-(C21-Pad2): track 11.8 -> 23.6 mm
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
Commit message: Add files via upload
Parts:
- removed J11, J16, J17, J18, J19, J1A1, J20, J3A1, J5, J6A1: Conn_01x01_Female, MountingHole:MountingHole_2.2mm_M2_ISO7380_Pad
- added J15: XLR3, Connector_Wire:SolderWire-0.25sqmm_1x03_P4.5mm_D0.65mm_OD2mm, F.Cu at (51.5, 40.0)
- added J21: XLR3, Connector_Wire:SolderWire-0.25sqmm_1x03_P4.5mm_D0.65mm_OD2mm, F.Cu at (51.0, 118.5)
- J2, J4: value Conn_01x01_Female -> XLR3; footprint MountingHole:MountingHole_2.2mm_M2_ISO7380_Pad -> Connector_Wire:SolderWire-0.25sqmm_1x03_P4.5mm_D0.65mm_OD2mm
- moved J4 82.3 mm to (78.0, 39.5)
- moved J2 12.0 mm to (78.0, 119.0)
Connections:
- J2 pad 1: ind -> V-R
- J4 pad 1: V- -> V-R
Routing:
- net V-: track 149.9 -> 193.2 mm
- net indR: track 127.1 -> 91.2 mm, vias 1 -> 0
- net V-R: track 154.9 -> 132.1 mm
- net /3: track 51.1 -> 29.5 mm
- net Net-(C17-Pad2): track 79.2 -> 58.9 mm
- net Net-(D8-A): track 58.3 -> 74.2 mm, vias 1 -> 0
- net Net-(D4-A): track 89.6 -> 75.7 mm, vias 0 -> 1
- net Net-(C4-Pad2): track 38.8 -> 26.9 mm
- net Net-(C14-Pad2): track 58.6 -> 49.8 mm
- net VCC: track 90.7 -> 98.3 mm, vias 1 -> 0
- net ind: track 74.8 -> 81.8 mm
- net /3A: track 28.6 -> 34.4 mm
- net VCCR: track 78.2 -> 73.9 mm, vias 0 -> 1
- net Net-(C9-Pad2): track 32.7 -> 36.4 mm
- net Net-(C10-Pad1): track 30.4 -> 27.6 mm, vias 0 -> 1
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