File: Highz-stereo.kicad_sch (KiCad schematic)
At the start: 79 parts, among them J1 Conn_01x01_Female, J10 Conn_01x01_Female, J11 Conn_01x01_Female, J12 Conn_01x01_Female, J13 Potmeter ground A, J14 potmeter ground B, J16 Conn_01x01_Female, J17 Conn_01x01_Female, J18 Conn_01x01_Female, J19 Conn_01x01_Female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

Commit message: Add files via upload
Parts:
- removed U1, U3: L7812CV, Package_TO_SOT_THT:TO-220-3_Vertical, symbol Regulator_Linear:L7812
- removed U2: OPA4134, Package_SO:SOIC-14_3.9x8.7mm_P1.27mm, symbol Amplifier_Operational:OPA4134
- added D1, D10: ZPD11, Diode_THT:D_DO-35_SOD27_P10.16mm_Horizontal, symbol Diode:ZPDxx
- added R1, R23: 100, Resistor_THT:R_Axial_DIN0204_L3.6mm_D1.6mm_P5.08mm_Horizontal, symbol Device:R
- added R27, R28: 150, Resistor_THT:R_Axial_DIN0204_L3.6mm_D1.6mm_P5.08mm_Horizontal, symbol Device:R
- added U2: OPA1679, Package_SO:SOIC-14_3.9x8.7mm_P1.27mm, symbol Amplifier_Operational:OPA1679
- C21, C22: value 0.33uF -> 680pF
- J13: value Potmeter ground A -> potmeter ground B
- J14: value potmeter ground B -> Potmeter ground A
Connections:
- net GND: now also D10.2 (A); no longer C21.2
- net GND1: now also J13.1 (Pin_1), D1.2 (A); no longer C22.2, J14.1 (Pin_1)
- net GNDA: now also J14.1 (Pin_1), U2.11 (V-); no longer J13.1 (Pin_1)
- net VCC: now also R23.1, U2.4 (V+)
- net VCCR: now also R1.1
- net ind: now also C21.1, U2.5 (+)
- net indR: now also C22.1, U2.12 (+)
- net at C6.2, R11.1, R7.2: now also U2.1
- net at C9.2, R13.1, R8.2: now also U2.7
- net at C6.1, R11.2, R9.2: now also U2.2 (-)
- net at R5.1, R6.1: now also D10.1 (K), R23.2; no longer C21.1
- net at D4.2 (A), D5.1 (K), J5.1 (Pin_1)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: now also R27.2, U2.3 (+)
- net at C9.1, R12.2, R13.2: now also U2.6 (-)
- net at R25.1, R26.1: now also D1.1 (K), R1.2; no longer C22.1
- net at C17.1, R20.2, R21.2: now also U2.13 (-)
- net at D8.2 (A), D9.1 (K), J17.1 (Pin_1)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: now also R28.2, U2.10 (+)
- net at C17.2, R21.1, R24.2: now also U2.14
- net at C14.1, R18.2, R19.2: now also U2.9 (-)
- net at C14.2, R19.1, R22.2: now also U2.8
- new net: C21.2, R27.1
- new net: C22.2, R28.1
Other:
- moved on the sheet: R14, R15, R3, R4

Commit message: Add files via upload
Parts:
- removed C18, C3: 33uF, Capacitor_THT:C_Disc_D5.0mm_W2.5mm_P2.50mm, symbol Device:C
- added C23, C3: 33uF, Capacitor_THT:CP_Radial_D5.0mm_P2.00mm, symbol Device:C_Polarized
- C11, C16, C19, C2, C20, C4, C5, C8: footprint Capacitor_THT:C_Disc_D5.0mm_W2.5mm_P2.50mm -> Capacitor_THT:C_Rect_L18.0mm_W9.0mm_P15.00mm_FKS3_FKP3
- C14, C17, C6, C9: footprint Capacitor_THT:C_Disc_D5.0mm_W2.5mm_P2.50mm -> Capacitor_THT:C_Rect_L7.2mm_W4.5mm_P5.00mm_FKS2_FKP2_MKS2_MKP2
- C21, C22: footprint Capacitor_THT:C_Disc_D5.0mm_W2.5mm_P2.50mm -> Capacitor_THT:C_Rect_L7.0mm_W4.5mm_P5.00mm
Connections:
- net GND: now also C23.2
- net GND1: now also C3.2
- net VCC: now also C23.1
- net VCCR: now also C3.1

Commit message: Add files via upload
Other:
- note added: "Suitable 4 gang potmeter PTD904-1015K-B103 if you want variable gain."
- note removed: "Suitable 2 gang potmeter P165M200PNN20MN103"
Changed lines of the file:
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@@
 		)
 	)
-	(text "Suitable 2 gang potmeter P165M200PNN20MN103"
+	(text "Suitable 4 gang potmeter PTD904-1015K-B103 if you want variable gain."
 		(exclude_from_sim no)
 		(at 89.916 133.858 0)

Commit message: Add files via upload
Parts:
- removed J11, J16, J17, J18, J19, J1A1, J2, J20, J3A1, J4, J5, J6A1: Conn_01x01_Female, MountingHole:MountingHole_2.2mm_M2_ISO7380_Pad, symbol double-gain-rescue:Conn_01x01_Female-Connector
- added J15, J2, J21, J4: XLR3, Connector_Wire:SolderWire-0.25sqmm_1x03_P4.5mm_D0.65mm_OD2mm, symbol Connector_Audio:XLR3
- C1, C13: mfr (none) -> TAP104K050SCS
- C10, C12, C15, C7: mfr (none) -> ECA-2AM470BJ
- C11, C16, C19, C2, C20, C4, C5, C8: mfr (none) -> B32522C0106K000
- C14, C17, C6, C9: mfr (none) -> FKP2O100471D00KSSD
- C21, C22: mfr (none) -> FKP2D006801D00KSSD
- C23, C3: mfr (none) -> 860010672011
- D1, D10: mfr (none) -> ZPD11
- D2, D3, D4, D5, D6, D7, D8, D9: mfr (none) -> 1N4148
- R1, R12, R18, R20, R23, R9: mfr (none) -> YR1B100RCC
- R10, R16, R17, R2: mfr (none) -> RNMF14FTC56K0
- R11, R13, R19, R21: mfr (none) -> RN60D4001FRE6
- R14, R15, R3, R4: mfr (none) -> RGP0207CHK1G0
- R22, R24, R7, R8: mfr (none) -> MFR-25FTE52-470R
- R25, R26, R5, R6: mfr (none) -> RNMF14FTC4K70
- R27, R28: mfr (none) -> RNF14FTD150R
- U2: mfr (none) -> OPA1679IDR
Connections:
- net 2: now also J4.2
- net 2A: now also J15.2
- net 3: now also J4.3
- net 3A: now also J15.3
- net GND1: now also J2.1, J4.1
- net GNDA: now also J15.1, J21.1
- net ind: now also J21.2
- net indR: now also J2.2
- net at D4.2 (A), D5.1 (K), R27.2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: now also J21.3
- net at D8.2 (A), D9.1 (K), R15.2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: now also J2.3
